Commit message: update moniarm description

File: moniarm_description/xacro/moniarm.ros2_control.xacro (robot description, xacro)
@@ -23,4 +23,11 @@
         <state_interface name="position"/>
       </joint>
+      <joint name="${prefix}joint3">
+        <command_interface name="position">
+          <param name="min">-1</param>
+          <param name="max">1</param>
+        </command_interface>
+        <state_interface name="position"/>
+      </joint>
     </ros2_control>
   </xacro:macro>

File: moniarm_description/xacro/moniarm_description.urdf.xacro (robot description, xacro)
@@ -5,7 +5,7 @@
   <xacro:property name="mass" value="1" /> <!-- arbitrary value for mass -->
   <xacro:property name="width" value="0.1" /> <!-- Square dimensions (widthxwidth) of beams -->
-  <xacro:property name="height1" value="2" /> <!-- Link 1 -->
-  <xacro:property name="height2" value="1" /> <!-- Link 2 -->
-  <xacro:property name="height3" value="1" /> <!-- Link 3 -->
+  <xacro:property name="height1" value="0.3" /> <!-- Link 1 -->
+  <xacro:property name="height2" value="0.45" /> <!-- Link 2 -->
+  <xacro:property name="height3" value="0.01" /> <!-- Link 3 -->
   <xacro:property name="camera_link" value="0.05" /> <!-- Size of square 'camera' box -->
   <xacro:property name="axel_offset" value="0.05" /> <!-- Space btw top of beam and the each joint -->
@@ -18,15 +18,15 @@
   <link name="${prefix}base_link">
     <collision>
-      <origin xyz="0 0 ${height1/2}" rpy="0 0 0"/>
-      <geometry>
+				<origin rpy="0 0 0" xyz="0 0 0" />
+				<geometry>
         <box size="${width} ${width} ${height1}"/>
       </geometry>
-    </collision>
+			</collision>
     <visual>
-      <origin xyz="0 0 ${height1/2}" rpy="0 0 0"/>
+      <origin xyz="-0.1 -0.15 0" rpy="89.5 0 1.5708"/>
       <geometry>
-        <box size="${width} ${width} ${height1}"/>
+					<mesh filename="package://moniarm_description/meshes/link1.stl" scale="0.005 0.005 0.005" />
       </geometry>
-      <material name="orange"/>
+      <material name="white"/>
     </visual>
     <inertial>
@@ -42,5 +42,5 @@
       <parent link="${prefix}base_link"/>
       <child link="${prefix}link1"/>
-      <origin xyz="0 ${width} ${height1 - axel_offset}" rpy="0 0 0"/>
+      <origin xyz="0 0 ${height1}" rpy="0 0 0"/>
       <axis xyz="0 1 0"/>
       <dynamics damping="0.7"/>
@@ -55,9 +55,10 @@
       </collision>
       <visual>
-        <origin xyz="0 0 ${height2/2 - axel_offset}" rpy="0 0 0"/>
+        <!-- <origin xyz="0.04 -0.45 0" rpy="0.01 -0.06 -0.01"/> -->
+        <origin xyz="-0.02 -0.1 -0.3" rpy="1.2 0 1.5708"/>
         <geometry>
-          <box size="${width} ${width} ${height2}"/>
+					<mesh filename="package://moniarm_description/meshes/link2.stl" scale="0.005 0.005 0.005" />
         </geometry>
-        <material name="yellow"/>
+        <material name="white"/>
       </visual>
       <inertial>
@@ -73,5 +74,5 @@
         <parent link="${prefix}link1"/>
         <child link="${prefix}link2"/>
-        <origin xyz="0 ${width} ${height2 - axel_offset*2}" rpy="0 0 0"/>
+        <origin xyz="0 0.01 ${height2}" rpy="0 0 0"/>
         <axis xyz="0 1 0"/>
         <dynamics damping="0.7"/>
@@ -82,13 +83,14 @@
           <origin xyz="0 0 ${height3/2 - axel_offset}" rpy="0 0 0"/>
           <geometry>
-            <box size="${width} ${width} ${height3}"/>
+            <box size="${width} ${width} ${height2}"/>
           </geometry>
         </collision>
         <visual>
-          <origin xyz="0 0 ${height3/2 - axel_offset}" rpy="0 0 0"/>
+          <!-- <origin xyz="-0.5 0 -0.45" rpy="1.2 0 1.5708"/> -->
+          <origin xyz="-0.64 -0.2 -0.4" rpy="2.1 0.1 1.5708"/>
           <geometry>
-            <box size="${width} ${width} ${height3}"/>
+            <mesh filename="package://moniarm_description/meshes/link3.stl" scale="0.005 0.005 0.005" />
           </geometry>
-          <material name="orange"/>
+          <material name="white"/>
         </visual>
         <inertial>
@@ -101,6 +103,6 @@
           </inertial>
         </link>
-        <joint name="${prefix}tool_joint" type="fixed">
-          <origin xyz="0 0 1" rpy="0 0 0" />
+        <joint name="${prefix}joint3" type="fixed">
+          <origin xyz="0 0 0.5" rpy="0 0 0" />
           <parent link="${prefix}link2"/>
           <child link="${prefix}tool_link" />
@@ -108,68 +110,26 @@
         <!-- Tool Link -->
         <link name="${prefix}tool_link">
-        </link>
-        <joint name="${prefix}hokuyo_joint" type="fixed">
-          <axis xyz="0 1 0" />
-          <origin xyz="0 0 ${height3 - axel_offset/2}" rpy="0 0 0"/>
-          <parent link="${prefix}link2"/>
-          <child link="${prefix}hokuyo_link"/>
-        </joint>
-        <!-- Hokuyo Laser -->
-        <link name="${prefix}hokuyo_link">
-          <collision>
-            <origin xyz="0 0 0" rpy="0 0 0"/>
-            <geometry>
-              <box size="0.1 0.1 0.1"/>
-            </geometry>
-          </collision>
-          <visual>
-            <origin xyz="0 0 0" rpy="0 0 0"/>
-            <geometry>
-              <mesh filename="package://moniarm_description/meshes/hokuyo.dae"/>
-            </geometry>
-          </visual>
-          <inertial>
-            <mass value="1e-5" />
-            <origin xyz="0 0 0" rpy="0 0 0"/>
-            <inertia ixx="1e-6" ixy="0" ixz="0" iyy="1e-6" iyz="0" izz="1e-6" />
+        <collision>
+          <origin xyz="0 0 ${height3/2 - axel_offset}" rpy="0 0 0"/>
+          <geometry>
+            <box size="${width} ${width} ${height2}"/>
+          </geometry>
+        </collision>
+        <visual>
+          <!-- <origin xyz="-0.55 -0.15 -1.13" rpy="1.57 0 1.5708"/> -->
+          <origin xyz="-0.435 -0.33 -1.13" rpy="1.57 0 1.5708"/>
+          <geometry>
+            <mesh filename="package://moniarm_description/meshes/link4.stl" scale="0.005 0.005 0.005" />
+          </geometry>
+          <material name="black"/>
+        </visual>
+        <inertial>
+          <origin xyz="0 0 ${height3/2 - axel_offset}" rpy="0 0 0"/>
+          <mass value="${mass}"/>
+          <inertia
+            ixx="${mass / 12.0 * (width*width + height3*height3)}" ixy="0.0" ixz="0.0"
+            iyy="${mass / 12.0 * (height3*height3 + width*width)}" iyz="0.0"
+            izz="${mass / 12.0 * (width*width + width*width)}"/>
           </inertial>
-        </link>
-        <joint name="${prefix}camera_joint" type="fixed">
-          <axis xyz="0 1 0" />
-          <origin xyz="${camera_link} 0 ${height3 - axel_offset*2}" rpy="0 0 0"/>
-          <parent link="${prefix}link2"/>
-          <child link="${prefix}camera_link"/>
-        </joint>
-        <!-- Camera -->
-        <link name="${prefix}camera_link">
-          <collision>
-            <origin xyz="0 0 0" rpy="0 0 0"/>
-            <geometry>
-              <box size="${camera_link} ${camera_link} ${camera_link}"/>
-            </geometry>
-          </collision>
-          <visual>
-            <origin xyz="0 0 0" rpy="0 0 0"/>
-            <geometry>
-              <box size="${camera_link} ${camera_link} ${camera_link}"/>
-            </geometry>
-            <material name="red"/>
-          </visual>
-          <inertial>
-            <mass value="1e-5" />
-            <origin xyz="0 0 0" rpy="0 0 0"/>
-            <inertia ixx="1e-6" ixy="0" ixz="0" iyy="1e-6" iyz="0" izz="1e-6" />
-          </inertial>
-        </link>
-        <!-- generate an optical frame http://www.ros.org/reps/rep-0103.html#suffix-frames
-        so that ros and opencv can operate on the camera frame correctly -->
-        <joint name="${prefix}camera_optical_joint" type="fixed">
-          <!-- these values have to be these values otherwise the gazebo camera image
-          won't be aligned properly with the frame it is supposedly originating from -->
-          <origin xyz="0 0 0" rpy="${-pi/2} 0 ${-pi/2}"/>
-          <parent link="${prefix}camera_link"/>
-          <child link="${prefix}camera_link_optical"/>
-        </joint>
-        <link name="${prefix}camera_link_optical">
         </link>
   </xacro:macro>

Commit message: moveit 4 link -> 5 link
1. Delete unused STLs
2. Remove urdf folder which is unsed
3. moveit 4 link -> 5 link in description.urdf.xacro

File: moniarm_description/xacro/moniarm.ros2_control.xacro (robot description, xacro)
@@ -30,4 +30,11 @@
         <state_interface name="position"/>
       </joint>
+      <joint name="${prefix}joint4">
+        <command_interface name="position">
+          <param name="min">-1</param>
+          <param name="max">1</param>
+        </command_interface>
+        <state_interface name="position"/>
+      </joint>
     </ros2_control>
   </xacro:macro>

File: moniarm_description/xacro/moniarm.urdf.xacro (robot description, xacro)
@@ -1,5 +1,5 @@
 <?xml version="1.0"?>
 <!-- Revolute-Revolute Manipulator -->
-<robot xmlns:xacro="http://www.ros.org/wiki/xacro" name="2dof_robot">
+<robot xmlns:xacro="http://www.ros.org/wiki/xacro" name="Moniarm">
   <xacro:arg name="prefix" default="" />
   <!-- Import moniarm macro -->
@@ -14,4 +14,10 @@
     <static>true</static>
   </gazebo>
+  <!-- World fixed joint-->
+  <joint name="world_fixed" type="fixed">
+    <origin xyz="0 0 0" rpy="0 0 0"/>
+    <parent link="world"/>
+    <child link="base_link"/>
+  </joint>
   <xacro:moniarm parent="world" prefix="$(arg prefix)">
     <origin xyz="0 0 0" rpy="0 0 0" />

File: moniarm_description/xacro/moniarm_description.urdf.xacro (robot description, xacro)
@@ -5,16 +5,42 @@
   <xacro:property name="mass" value="1" /> <!-- arbitrary value for mass -->
   <xacro:property name="width" value="0.1" /> <!-- Square dimensions (widthxwidth) of beams -->
-  <xacro:property name="height1" value="0.3" /> <!-- Link 1 -->
-  <xacro:property name="height2" value="0.45" /> <!-- Link 2 -->
+  <xacro:property name="height1" value="0.01" /> <!-- Link 1 -->
+  <xacro:property name="height2" value="0.01" /> <!-- Link 2 -->
   <xacro:property name="height3" value="0.01" /> <!-- Link 3 -->
+  <xacro:property name="height3" value="0.01" /> <!-- Link 4 -->
+  <xacro:property name="height3" value="0.01" /> <!-- Link 5 -->
   <xacro:property name="camera_link" value="0.05" /> <!-- Size of square 'camera' box -->
   <xacro:property name="axel_offset" value="0.05" /> <!-- Space btw top of beam and the each joint -->
-  <joint name="${prefix}base_joint" type="fixed">
-    <xacro:insert_block name="origin" />
-    <parent link="${parent}"/>
-    <child link="${prefix}base_link" />
+  <!-- Base Link -->
+  <link name="base_link">
+      <collision>
+          <origin xyz="0 0 0" rpy="0 0 0"/>
+          <geometry>
+              <mesh filename="package://moniarm_description/meshes/base.stl" scale="0.005 0.005 0.005"/>
+          </geometry>
+      </collision>
+      <visual>
+          <origin xyz="0 0 0" rpy="1.5708 0 0"/>
+          <geometry>
+              <mesh filename="package://moniarm_description/meshes/base.stl" scale="0.005 0.005 0.005"/>
+          </geometry>
+          <material name="grey"/>
+      </visual>
+      <inertial>
+          <origin xyz="0 0 0" rpy="0 0 0"/>
+          <mass value="1"/>
+          <inertia ixx="1.0" ixy="0.0" ixz="0.0" iyy="1.0" iyz="0.0" izz="1.0"/>
+      </inertial>
+  </link>
+  <!-- Joint 1, motor0 -->
+  <joint name="${prefix}joint1" type="continuous">
+    <parent link="${prefix}base_link"/>
+    <child link="${prefix}link1"/>
+    <origin xyz="0 0 ${height1}" rpy="0 0 0"/>
+    <axis xyz="0 1 0"/>
+    <dynamics damping="0.7"/>
   </joint>
-  <!-- Base Link -->
-  <link name="${prefix}base_link">
+  <!-- Link 1-->
+  <link name="${prefix}link1">
     <collision>
 				<origin rpy="0 0 0" xyz="0 0 0" />
@@ -24,5 +50,5 @@
 			</collision>
     <visual>
-      <origin xyz="-0.1 -0.15 0" rpy="89.5 0 1.5708"/>
+      <origin xyz="0.06 -0.12 0.17" rpy="0 0 -1.5708"/>
       <geometry>
 					<mesh filename="package://moniarm_description/meshes/link1.stl" scale="0.005 0.005 0.005" />
@@ -39,13 +65,14 @@
       </inertial>
     </link>
-    <joint name="${prefix}joint1" type="continuous">
-      <parent link="${prefix}base_link"/>
-      <child link="${prefix}link1"/>
-      <origin xyz="0 0 ${height1}" rpy="0 0 0"/>
+    <!-- Joint 2, motor1 -->
+    <joint name="${prefix}joint2" type="continuous">
+      <parent link="${prefix}link1"/>
+      <child link="${prefix}link2"/>
+      <origin xyz="0 0.01 ${height2}" rpy="0 0 0"/>
       <axis xyz="0 1 0"/>
       <dynamics damping="0.7"/>
     </joint>
-    <!-- Middle Link -->
-    <link name="${prefix}link1">
+    <!-- Link 2-->
+    <link name="${prefix}link2">
       <collision>
         <origin xyz="0 0 ${height2/2 - axel_offset}" rpy="0 0 0"/>
@@ -55,6 +82,5 @@
       </collision>
       <visual>
-        <!-- <origin xyz="0.04 -0.45 0" rpy="0.01 -0.06 -0.01"/> -->
-        <origin xyz="-0.02 -0.1 -0.3" rpy="1.2 0 1.5708"/>
+        <origin xyz="-0.02 -0.1 -0.02" rpy="1.2 -0.1 0"/>
         <geometry>
 					<mesh filename="package://moniarm_description/meshes/link2.stl" scale="0.005 0.005 0.005" />
@@ -71,13 +97,14 @@
         </inertial>
       </link>
-      <joint name="${prefix}joint2" type="continuous">
-        <parent link="${prefix}link1"/>
-        <child link="${prefix}link2"/>
+      <!-- Joint 3, motor2 -->
+      <joint name="${prefix}joint3" type="continuous">
+        <parent link="${prefix}link2"/>
+        <child link="${prefix}link3"/>
         <origin xyz="0 0.01 ${height2}" rpy="0 0 0"/>
         <axis xyz="0 1 0"/>
         <dynamics damping="0.7"/>
       </joint>
-      <!-- Top Link -->
-      <link name="${prefix}link2">
+      <!-- Link 3 -->
+      <link name="${prefix}link3">
         <collision>
           <origin xyz="0 0 ${height3/2 - axel_offset}" rpy="0 0 0"/>
@@ -87,10 +114,9 @@
         </collision>
         <visual>
-          <!-- <origin xyz="-0.5 0 -0.45" rpy="1.2 0 1.5708"/> -->
-          <origin xyz="-0.64 -0.2 -0.4" rpy="2.1 0.1 1.5708"/>
+          <origin xyz="-0.02 -0.1 0.0" rpy="1.2 0.3 0"/>
           <geometry>
             <mesh filename="package://moniarm_description/meshes/link3.stl" scale="0.005 0.005 0.005" />
           </geometry>
-          <material name="white"/>
+          <material name="green"/>
         </visual>
         <inertial>
@@ -103,11 +129,12 @@
           </inertial>
         </link>
-        <joint name="${prefix}joint3" type="fixed">
+        <!-- Joint 4, motor3 -->
+        <joint name="${prefix}joint4" type="continuous">
           <origin xyz="0 0 0.5" rpy="0 0 0" />
-          <parent link="${prefix}link2"/>
-          <child link="${prefix}tool_link" />
+          <parent link="${prefix}link3"/>
+          <child link="${prefix}link4" />
         </joint>
-        <!-- Tool Link -->
-        <link name="${prefix}tool_link">
+          <!-- Link 4, motor+link+pump -->
+        <link name="${prefix}link4">
         <collision>
           <origin xyz="0 0 ${height3/2 - axel_offset}" rpy="0 0 0"/>
@@ -117,10 +144,9 @@
         </collision>
         <visual>
-          <!-- <origin xyz="-0.55 -0.15 -1.13" rpy="1.57 0 1.5708"/> -->
-          <origin xyz="-0.435 -0.33 -1.13" rpy="1.57 0 1.5708"/>
+          <origin xyz="0 0 0" rpy="0 0 0"/>
           <geometry>
             <mesh filename="package://moniarm_description/meshes/link4.stl" scale="0.005 0.005 0.005" />
           </geometry>
-          <material name="black"/>
+          <material name="green"/>
         </visual>
         <inertial>
